File: Interface.kicad_sch (KiCad schematic)
At the start: 10 parts, among them SW1 RotaryEncoder_Switch, SW2 RotaryEncoder_Switch

Commit message: Update 1/29/25
Changed lines of the file:
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@@
 (kicad_sch
-	(version 20231120)
+	(version 20241004)
 	(generator "eeschema")
-	(generator_version "7.99")
+	(generator_version "8.99")
 	(paper "A4")
 	(junction
