File: PSUMonitoring.kicad_sch (KiCad schematic)
At the start: 47 parts, among them Q1 Q_Dual_NMOS_G1S2G2D2S1D1, Q2 Q_Dual_NMOS_G1S2G2D2S1D1, Q3 Q_Dual_NMOS_G1S2G2D2S1D1, Q4 Q_Dual_NMOS_G1S2G2D2S1D1, U1 LM321, U2 ADS131M02, X1 ASCO

Commit message: Update 1/29/25
Changed lines of the file:
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@@
 (kicad_sch
-	(version 20231120)
+	(version 20241004)
 	(generator "eeschema")
-	(generator_version "7.99")
+	(generator_version "8.99")
 	(paper "A4")
 	(junction
