File: ProgSupply.kicad_sch (KiCad schematic)
At the start: 7 parts, among them J3 USB_C_Receptacle_USB2.0, U8 D3V3XA4B10LP

Commit message: Update 1/29/25
Parts:
- removed C21, C22: 1uF, symbol Device:C_Small
- removed FB1: 100R @ 100 MHz, symbol Device:FerriteBead_Small
Connections:
- net VBUS: now also F1.2
