File: system_power.kicad_sch (KiCad schematic)
At the start: 19 parts, among them U4 TPS56339DDC, U5 TLV73333PDBV, U6 TLV73333PDBV

Commit message: Update 1/29/25
Changed lines of the file:
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@@
 (kicad_sch
-	(version 20231120)
+	(version 20241004)
 	(generator "eeschema")
-	(generator_version "7.99")
+	(generator_version "8.99")
 	(paper "A4")
 	(junction
